Commit message: Make frcrobot_description base_link z=floor height to match assumption in 2019_compbot.urdf file

File: zebROS_ws/src/frcrobot_description/urdf/frcrobot.xacro (robot description, xacro)
@@ -7,4 +7,5 @@
 	<xacro:property name="base_depth" value=".75" />
 	<xacro:property name="swerve_box_size" value=".075" />
+	<xacro:property name="wheel_diameter" value=".0675" />
 	<xacro:macro name="swerve_module" params="prefix x y">
 		<link name="${prefix}_angle">
@@ -22,5 +23,5 @@
 			<visual>
 				<geometry>
-					<cylinder length=".04" radius=".0675"/>
+					<cylinder length=".04" radius="${wheel_diameter}"/>
 				</geometry>
 				<origin xyz="0 0 0" rpy="${pi/2} 0 0"/>
@@ -31,5 +32,5 @@
 		</link>
 		<joint name="base_to_${prefix}_angle" type="continuous">
-			<parent link="base_link"/>
+			<parent link="base_plate"/>
 			<child link="${prefix}_angle"/>
 			<origin xyz="${x} ${y} -${base_height/2}" rpy="0 0 0"/>
@@ -38,5 +39,5 @@
 			<parent link="${prefix}_angle"/>
 			<child link="${prefix}_speed"/>
-			<origin xyz="0 0 -0.0675" rpy="0 0 0"/>
+			<origin xyz="0 0 -${wheel_diameter}" rpy="0 0 0"/>
 		</joint>
 	</xacro:macro>
@@ -54,11 +55,12 @@
 		<parent link="base_link"/>
 		<child link="base_plate"/>
-		<origin xyz="0 0 0 " rpy="0 0 0"/>
+		<origin xyz="0 0 ${wheel_diameter + base_height/2}" rpy="0 0 0"/>
 	</joint>
 	<xacro:property name="elevator_height" value="1.1" />
+	<xacro:property name="elevator_width"  value="${base_width / 2.}" />
 	<link name="elevator_plate">
 		<visual>
 			<geometry>
-				<box size="${base_width * 2. / 3.} 0.05 ${elevator_height}"/>
+				<box size="${elevator_width} 0.05 ${elevator_height}"/>
 			</geometry>
 			<material name="yellow">
@@ -68,5 +70,5 @@
 	</link>
 	<joint name="elevator_plate_to_base_link" type="fixed">
-		<parent link="base_link"/>
+		<parent link="base_plate"/>
 		<child link="elevator_plate"/>
 		<origin xyz="-0.25 0 ${elevator_height/2 + base_height/2}" rpy="0 0 ${pi/2}"/>
