Commit message: Hook up transform to attach rs t265 to comp robot tf tree

File: zebROS_ws/src/controller_node/urdf/2019_compbot.urdf (robot description, URDF)
Before this commit: robot 2019_compbot, 10 links, 9 joints
Links:
- added link camera_pose_frame
Joints:
- added joint camera_joint: type fixed, parent camera_pose_frame, child base_link, origin xyz=1.04 0 0.216 rpy=0 -1.57 0

Commit message: Fix orienation of t265 camera in urdf

File: zebROS_ws/src/controller_node/urdf/2019_compbot.urdf (robot description, URDF)
Before this commit: robot 2019_compbot, 11 links, 10 joints
Joints:
- joint camera_joint: origin xyz=1.04 0 0.216 rpy=0 -1.57 0 -> xyz=0.216 0.0 1.04 rpy=0 0 0

Commit message: Fix origin coords of t265 camera in urdf

File: zebROS_ws/src/controller_node/urdf/2019_compbot.urdf (robot description, URDF)
Before this commit: robot 2019_compbot, 11 links, 10 joints
Joints:
- joint camera_joint: origin xyz=0.216 0.0 1.04 rpy=0 0 0 -> xyz=-0.216 0.0 1.04 rpy=0 0 0

Commit message: More work on urdf robot model

File: zebROS_ws/src/controller_node/urdf/2019_compbot.urdf (robot description, URDF)
Before this commit: robot 2019_compbot, 11 links, 10 joints
Joints:
- joint camera_joint: child base_link -> camera_pose_frame; parent camera_pose_frame -> base_link

File: zebROS_ws/src/frcrobot_description/urdf/frcrobot.xacro (robot description, xacro)
@@ -13,7 +13,7 @@
 					<box size="${swerve_box_size} ${swerve_box_size} ${swerve_box_size}"/>
 				</geometry>
-				<origin xyz="0 0 0" rpy="0 0 0"/>
+				<origin xyz="0 0 -${swerve_box_size / 2}" rpy="0 0 0"/>
 				<material name="red">
-					<color rgba="1 0 0 1"/>
+					<color rgba="1 0 0 .5"/>
 				</material>
 			</visual>
@@ -24,5 +24,5 @@
 					<cylinder length=".04" radius=".0675"/>
 				</geometry>
-				<origin xyz="${x} ${y} -${base_height/2 + swerve_box_size}" rpy="${pi/2} 0 0"/>
+				<origin xyz="0 0 0" rpy="${pi/2} 0 0"/>
 				<material name="black">
 					<color rgba="0 0 0 1"/>
@@ -33,13 +33,13 @@
 			<parent link="base_link"/>
 			<child link="${prefix}_angle"/>
-			<origin xyz="${x} ${y} -${base_height/2 + swerve_box_size/2}" rpy="0 0 0"/>
+			<origin xyz="${x} ${y} -${base_height/2}" rpy="0 0 0"/>
 		</joint>
 		<joint name="${prefix}_angle_to_speed" type="continuous">
 			<parent link="${prefix}_angle"/>
 			<child link="${prefix}_speed"/>
-			<origin xyz="0 0 0" rpy="0 0 0"/>
+			<origin xyz="0 0 -0.0675" rpy="0 0 0"/>
 		</joint>
 	</xacro:macro>
-	<link name="base_link">
+	<link name="base_plate">
 		<visual>
 			<geometry>
@@ -51,7 +51,29 @@
 		</visual>
 	</link>
+	<joint name="base_plate_to_base_link" type="fixed">
+		<parent link="base_link"/>
+		<child link="base_plate"/>
+		<origin xyz="0 0 0 " rpy="0 0 0"/>
+	</joint>
+	<xacro:property name="elevator_height" value="1.1" />
+	<link name="elevator_plate">
+		<visual>
+			<geometry>
+				<box size="${base_width * 2. / 3.} 0.05 ${elevator_height}"/>
+			</geometry>
+			<material name="yellow">
+				<color rgba="1 1 0 1"/>
+			</material>
+		</visual>
+	</link>
+	<joint name="elevator_plate_to_base_link" type="fixed">
+		<parent link="base_link"/>
+		<child link="elevator_plate"/>
+		<origin xyz="-0.25 0 ${elevator_height/2 + base_height/2}" rpy="0 0 ${pi/2}"/>
+	</joint>
 	<xacro:swerve_module prefix="lf" x="${base_width/2 - swerve_box_size/2}" y="${base_depth/2 - swerve_box_size/2}"/>
 	<xacro:swerve_module prefix="rf" x="${base_width/2 - swerve_box_size/2}" y="-${base_depth/2 - swerve_box_size/2}"/>
 	<xacro:swerve_module prefix="lr" x="-${base_width/2 - swerve_box_size/2}" y="${base_depth/2 - swerve_box_size/2}"/>
 	<xacro:swerve_module prefix="rr" x="-${base_width/2 - swerve_box_size/2}" y="-${base_depth/2 - swerve_box_size/2}"/>
+	<xacro:include filename="$(find controller_node)/urdf/2019_compbot.urdf"/>
 </robot>

Commit message: Basics of getting simple robot model into gazebo

File: zebROS_ws/src/controller_node/urdf/2019_compbot.urdf (robot description, URDF)
Before this commit: robot 2019_compbot, 11 links, 10 joints
Joints:
- joint imu_link_joint: type floating -> fixed

File: zebROS_ws/src/frcrobot_description/frcrobot_description/urdf/frcrobot.xacro (robot description, xacro)
@@ -19,4 +19,14 @@
 				</material>
 			</visual>
+			<collision>
+				<origin xyz="0 0 -${swerve_box_size / 2}" rpy="0 0 0"/>
+				<geometry>
+					<box size="${swerve_box_size} ${swerve_box_size} ${swerve_box_size}"/>
+				</geometry>
+			</collision>
+			<inertial>
+				<mass value="0.5"/>
+				<inertia ixx="0.1" iyy="0.1" izz="0.1" ixy="0.0" ixz="0.0" iyz="0.0"/>
+			</inertial>
 		</link>
 		<link name="${prefix}_speed">
@@ -30,4 +40,14 @@
 				</material>
 			</visual>
+			<collision>
+				<origin xyz="0 0 0" rpy="${pi/2} 0 0"/>
+				<geometry>
+					<cylinder length=".04" radius="${wheel_diameter}"/>
+				</geometry>
+			</collision>
+			<inertial>
+				<mass value="0.5"/>
+				<inertia ixx="0.1" iyy="0.1" izz="0.1" ixy="0.0" ixz="0.0" iyz="0.0"/>
+			</inertial>
 		</link>
 		<joint name="base_to_${prefix}_angle" type="continuous">
@@ -35,4 +55,5 @@
 			<child link="${prefix}_angle"/>
 			<origin xyz="${x} ${y} -${base_height/2}" rpy="0 0 0"/>
+			<axis xyz="0 0 1" />
 		</joint>
 		<joint name="${prefix}_angle_to_speed" type="continuous">
@@ -40,4 +61,5 @@
 			<child link="${prefix}_speed"/>
 			<origin xyz="0 0 -${wheel_diameter}" rpy="0 0 0"/>
+			<axis xyz="0 1 0" />
 		</joint>
 	</xacro:macro>
@@ -51,4 +73,13 @@
 			</material>
 		</visual>
+		<collision>
+			<geometry>
+				<box size="${base_width} ${base_depth} ${base_height}"/>
+			</geometry>
+		</collision>
+		<inertial>
+		  <mass value="10.0"/>
+		  <inertia ixx="1.0" iyy="1.0" izz="1.0" ixy="0.0" ixz="0.0" iyz="0.0"/>
+		</inertial>
 	</link>
 	<joint name="base_plate_to_base_link" type="fixed">

Commit message: one or two hacky fixes to get auto align working

File: zebROS_ws/src/controller_node/urdf/2019_compbot.urdf (robot description, URDF)
Before this commit: robot 2019_compbot, 11 links, 10 joints
Joints:
- joint zed_camera_center_joint: origin xyz=-0.234 -0.1576 1.1684 rpy=0 0 0 -> xyz=0.006589 -0.234 1.1684 rpy=0 0 0

Commit message: changed ZED transforms

File: zebROS_ws/src/controller_node/urdf/2019_compbot.urdf (robot description, URDF)
Before this commit: robot 2019_compbot, 11 links, 10 joints
Joints:
- joint zed_camera_center_joint: origin xyz=0.006589 -0.234 1.1684 rpy=0 0 0 -> xyz=0.006589 -0.474 1.1684 rpy=0 0 0

Commit message: updated transforms

File: zebROS_ws/src/controller_node/urdf/2019_compbot.urdf (robot description, URDF)
Before this commit: robot 2019_compbot, 11 links, 10 joints
Joints:
- joint zed_camera_center_joint: origin xyz=0.006589 -0.474 1.1684 rpy=0 0 0 -> xyz=-0.304589 -0.532 1.1684 rpy=0 0 0

Commit message: transforms

File: zebROS_ws/src/controller_node/urdf/2019_compbot.urdf (robot description, URDF)
Before this commit: robot 2019_compbot, 11 links, 10 joints
Joints:
- joint zed_camera_center_joint: origin xyz=-0.304589 -0.532 1.1684 rpy=0 0 0 -> xyz=-0.304589 -0.570 1.1684 rpy=0 0 0

Commit message: transforms, record files, teleop parameters

File: zebROS_ws/src/controller_node/urdf/2019_compbot.urdf (robot description, URDF)
Before this commit: robot 2019_compbot, 11 links, 10 joints
Joints:
- joint zed_camera_center_joint: origin xyz=-0.304589 -0.570 1.1684 rpy=0 0 0 -> xyz=-0.304589 -0.515 1.1684 rpy=0 0 0

Commit message: added sleep in align_server, increased place cmd_vel, transforms, record

File: zebROS_ws/src/controller_node/urdf/2019_compbot.urdf (robot description, URDF)
Before this commit: robot 2019_compbot, 11 links, 10 joints
Joints:
- joint zed_camera_center_joint: origin xyz=-0.304589 -0.515 1.1684 rpy=0 0 0 -> xyz=-0.304589 -0.532 1.1684 rpy=0 0 0

Commit message: updates to zed urdf

File: zebROS_ws/src/controller_node/urdf/2019_compbot.urdf (robot description, URDF)
Before this commit: robot 2019_compbot, 11 links, 10 joints
Joints:
- joint zed_camera_center_joint: origin xyz=-0.304589 -0.532 1.1684 rpy=0 0 0 -> xyz=-0.434589 -0.532 1.1684 rpy=0 0 0

Commit message: Reverse child<->parent in realsense to base_link tf (#27)

File: zebROS_ws/src/controller_node/urdf/2019_compbot.urdf (robot description, URDF)
Before this commit: robot 2019_compbot, 11 links, 10 joints
Links:
- removed link camera_pose_frame
- added link rs_t265_pose_frame
Joints:
- removed joint camera_joint
- added joint rs_t265_joint: type fixed, parent rs_t265_pose_frame, child base_link, origin xyz=0.216 0.0 -1.04 rpy=0 0 0
