Commit message: Swap rotation on intake tf frame

File: zebROS_ws/src/controller_node/urdf/2021_compbot.xacro (robot description, xacro)
@@ -12,5 +12,5 @@
         <parent link="base_link"/>
         <child link="intake"/>
-        <origin xyz="-0.6332 0.0 0.0" rpy="0 0 3.14159265" />
+        <origin xyz="-0.6332 0.0 0.0" rpy="0 0 0" />
     </joint>
 </robot>

Commit message: Assorted improvements to galactic search

File: zebROS_ws/src/controller_node/urdf/2021_compbot.xacro (robot description, xacro)
@@ -12,5 +12,5 @@
         <parent link="base_link"/>
         <child link="intake"/>
-        <origin xyz="-0.6332 0.0 0.0" rpy="0 0 0" />
+        <origin xyz="0.6332 0.0 0.0" rpy="0 0 0"/>
     </joint>
 </robot>
