Commit message: 20220302 prep (#65)
* Prep for Wed meeting

Initial attempt at climber arm scaling factor
Replace stub of wpi::GetStackTrace with actual code
Delay for ctre read threads based on array index rather than can ID
Split up frc robot interface for hopefully quicker builds

* Don't run an additional copy of the imu zero code in teleop

* Various transforms added
Zed config setup for object detection code

* Enable falcon encoders for 2022 test setup
Set climber conversion factor for test setup
Remove fake talons from hardware interface

File: zebROS_ws/src/controller_node/urdf/2022_compbot.xacro (robot description, xacro)
@@ -1,5 +1,11 @@
 <?xml version="1.0"?>
-<robot name="2021_compbot" xmlns:xacro="http://ros.org/wiki/xacro">
+<robot name="2022_compbot" xmlns:xacro="http://ros.org/wiki/xacro">
     <link name="base_link"/>
     <!-- add important transforms for 2022 -->
+    <link name="intake"/>
+    <joint name="intake_joint" type="fixed">
+        <parent link="base_link"/>
+        <child link="intake"/>
+        <origin xyz="0.6561 0.0 0.210" rpy="0 0 0"/>
+    </joint>
 </robot>
