Commit message: Arm server (#124)
* add minifrc stls

* Added action file for the arm

* Added the controller for the arm, and started on the action server and client (Also fixed some stuff with simlaunch but yea)

* I think this should be everything for the action server except the code that actually moves the motor, I'll figure that out next meeting

* added some to the movey part

* I think this should be pretty much done :D

* A bit of debugging

* test push

* oopsies two file deleted one renamed the other

* modified the arm server and actionfile

* Fixed some issues with the code

* Some changes

* I think everything is finished. There are definitely some errors but I'm just not sure how to fix it

* 'Fix bug, find another one, repeat' - This code (For realisies though its almost done)

* ITS FINALLY DONE, WOOO

* Cleaned up the code to get rid of testing stuff (I forgot to before)

* Cleaned up some stuff that Ben pointed out (thanks :D), and I made A LOT more comments explaining the code (or at least they should explain it correctly) for future students (And myself but we won't talk about that lol)

---------

Co-authored-by: BenBean18 <beakerthespeaker@gmail.com>
Co-authored-by: Adele McS <adelemcshane@adeles-air.lan>
Co-authored-by: Adele McS <adelemcshane@Adeles-MacBook-Air.local>

File: zebROS_ws/src/minifrcrobot_description/urdf/robot.urdf (robot description, URDF)
Before this commit: robot onshape, 21 links, 20 joints
Links:
- removed link babys_first_orchestra_link
- removed link candle1_link
- removed link pigeon2_link
- removed link robot_code_ready_link
- added link robot_code_ready_jetson_link
Joints:
- removed joint babys_first_orchestra
- removed joint candle1
- removed joint pigeon2
- joint robot_code_ready_jetson: child robot_code_ready_link -> robot_code_ready_jetson_link
