Commit message: update field urdf to include robot stl

File: zebROS_ws/src/frcrobot_description/frcrobot_description/urdf/2024_field.urdf (robot description, URDF)
Before this commit: robot field, 2 links, 1 joints
Links:
- added link apollo_link; visual mesh filename=package://frcrobot_description/meshes/2024_compbot.stl
Joints:
- added joint base_link_to_apollo: type floating, parent base_link, child apollo_link, origin xyz=0 0 0 rpy=1.57 3.14 -1.57
